File: pcb/010.sch (KiCad schematic (older format))
At the start: 11 parts, among them J1 CONN_12, SW1 ap, SW2 so, SW3 ei, SW4 tn, SW5 spcsh

Commit message: readme
Parts:
- J1: footprint SF_Connectors:1X12 -> Pin_Headers:Pin_Header_Straight_1x12_Pitch2.54mm
Changed lines of the file:
@@
 F 0 "J1" H 4822 3105 45  0000 R CNN
 F 1 "CONN_12" H 4822 3189 45  0000 R CNN
-F 2 "SF_Connectors:1X12" H 5100 3950 20  0001 C CNN
+F 2 "Pin_Headers:Pin_Header_Straight_1x12_Pitch2.54mm" H 5100 3950 20  0001 C CNN
 F 3 "" H 5100 2650 50  0001 C CNN
 F 4 "XXX-00000" H 4822 3284 60  0000 R CNN "Field4"
